Commit message: Update simulation: improve manual and arm control

File: robot_workspace/x3plus_ws/src/x3plus_multi_bringup/urdf/yahboomcar_X3plus.urdf.xacro (robot description, xacro)
@@ -15,4 +15,13 @@
     <material name="White">
         <color rgba="0.7 0.7 0.7 1"/>
+    </material>
+    <material name="Black">
+        <color rgba="0.2 0.2 0.2 1"/>
+    </material>
+    <material name="Red">
+        <color rgba="1 0 0 1"/>
+    </material>
+    <material name="DarkGray">
+        <color rgba="0.3 0.3 0.3 1"/>
     </material>
     <link name="${prefix}${ns}base_footprint"/>
@@ -96,5 +105,5 @@
         </inertial>
     </xacro:common_link>
-    <xacro:fixed_joint name="camera_joint" parent="base_link" child="camera_link" xyz="-0.043645 0 0.41955" rpy="0 0 0"/>
+    <xacro:fixed_joint name="camera_joint" parent="base_link" child="camera_link" xyz="0.043645 0 0.41955" rpy="0 0 0"/>
     <xacro:common_link name="arm_link1" material="White" path="X3plus">
         <inertial>
@@ -259,5 +268,5 @@
         </inertial>
     </xacro:common_link>
-    <xacro:fixed_joint name="mono_joint" parent="arm_link4" child="mono_link" xyz="-0.0481 -0.05145 -0.0022"
+    <xacro:fixed_joint name="mono_joint" parent="arm_link4" child="mono_link" xyz="0.0481 -0.05145 -0.0022"
                  rpy="${pi/2} 0 0"/>
     <xacro:yahboomcar_X3plus_ros2_control

File: robot_workspace/x3plus_ws/src/x3plus_sim_bringup/urdf/yahboomcar_X3plus.urdf.xacro (robot description, xacro)
@@ -6,4 +6,13 @@
     <material name="White">
         <color rgba="0.7 0.7 0.7 1"/>
+    </material>
+    <material name="Black">
+        <color rgba="0.2 0.2 0.2 1"/>
+    </material>
+    <material name="Red">
+        <color rgba="1 0 0 1"/>
+    </material>
+    <material name="DarkGray">
+        <color rgba="0.3 0.3 0.3 1"/>
     </material>
     <xacro:property name="ns" value="$(arg ns)"/>
@@ -72,5 +81,5 @@
     <fixed_joint name="base_joint" parent="base_footprint" child="base_link" xyz="0.0 0.0 0.076" rpy="0 0 0"/>
     <fixed_joint name="base_imu" parent="base_link" child="imu_link" xyz="0.001 0.017 0.0322" rpy="0 3.1415 1.5707"/>
-    <common_link name="laser_link" material="White" path="sensor">
+    <common_link name="laser_link" material="White" path="sensor_X3plus">
         <inertial>
             <origin xyz="-0.0176558922685589 0.000671805271544437 0.0219302095894866" rpy="0 0 0"/>
@@ -81,5 +90,5 @@
     </common_link>
     <fixed_joint name="laser_joint" parent="base_link" child="laser_link" xyz="0.10478 0 0.0471" rpy="0 0 0"/>
-    <common_link name="camera_link" material="White" path="sensor">
+    <common_link name="camera_link" material="White" path="sensor_X3plus">
         <inertial>
             <origin xyz="0 0 0" rpy="0 0 0"/>
@@ -88,5 +97,5 @@
         </inertial>
     </common_link>
-    <fixed_joint name="camera_joint" parent="base_link" child="camera_link" xyz="-0.043645 0 0.41955" rpy="0 0 0"/>
+    <fixed_joint name="camera_joint" parent="base_link" child="camera_link" xyz="0.043645 0 0.41955" rpy="0 0 0"/>
     <common_link name="arm_link1" material="White" path="X3plus">
         <inertial>
@@ -243,5 +252,5 @@
     <continuous_joint name="llink_joint3" parent="arm_link5" child="llink3" xyz="-0.0035 0.0045 -0.0505"
                       rpy="0 -${pi/2} 0" mimic="-1"/>
-    <common_link name="mono_link" material="White" path="sensor">
+    <common_link name="mono_link" material="White" path="sensor_X3plus">
         <inertial>
             <origin xyz="5.8458E-05 0.0095015 -0.0014824" rpy="0 0 0"/>
@@ -251,5 +260,5 @@
         </inertial>
     </common_link>
-    <fixed_joint name="mono_joint" parent="arm_link4" child="mono_link" xyz="-0.0481 -0.05145 -0.0022"
+    <fixed_joint name="mono_joint" parent="arm_link4" child="mono_link" xyz="0.0481 -0.05145 -0.0022"
                  rpy="${pi/2} 0 0"/>
 </robot>
