Commit message: Update simulation: improve manual and arm control

File: robot_workspace/x3plus_ws/src/yahboomcar_description/urdf/yahboomcar_X3plus.urdf.xacro (robot description, xacro)
@@ -1,16 +1,33 @@
 <?xml version="1.0" encoding="utf-8"?>
 <robot name="yahboomcar_X3plus" xmlns:xacro="http://wiki.ros.org/xacro">
-    <material name="Green">
-        <color rgba="0 0.7 0 1"/>
+    <!-- Material Definitions -->
+    <material name="Black">
+        <color rgba="0.0 0.0 0.0 1.0"/>
     </material>
     <material name="White">
-        <color rgba="0.7 0.7 0.7 1"/>
+        <color rgba="0.95 0.95 0.95 1.0"/>
     </material>
+    <material name="Green">
+        <color rgba="0.0 0.5 0.0 1.0"/>
+    </material>
+    <material name="Red">
+        <color rgba="1.0 0.0 0.0 1.0"/>
+    </material>
+    <material name="DarkGray">
+        <color rgba="0.3 0.3 0.3 1.0"/>
+    </material>
+    <!-- XACRO Argument: Robot namespace for multi-robot support -->
+    <!-- Default: empty string (no namespace prefix) for single robot -->
+    <!-- Usage: xacro file.xacro ns:=robot1/ (for multi-robot with slash at end) -->
+    <xacro:arg name="ns" default=""/>  <!-- Default empty namespace -->
+    <!-- Helper wheel cylinders are useful for debugging wheel kinematics, but can clutter RViz. -->
+    <xacro:arg name="show_helper_wheels" default="false"/>
     <xacro:property name="ns" value="$(arg ns)"/>
-    <link name="${ns}/base_footprint"/>
-    <link name="${ns}/imu_link"/>
+    <xacro:property name="show_helper_wheels" value="$(arg show_helper_wheels)"/>
+    <link name="base_footprint"/>
+    <link name="imu_link"/>
     <!-- common link-->
     <xacro:macro name="common_link" params="name material path *origin">
-        <link name="${ns}/${name}">
+        <link name="${name}">
             <visual>
                 <geometry>
@@ -57,5 +74,61 @@
         </joint>
     </xacro:macro>
-    <common_link name="${ns}/base_link" material="Green" path="X3plus">
+    <!-- ==================== WHEEL LINKS AND JOINTS MACROS ==================== -->
+    <!-- CONFIGURABLE WHEEL PARAMETERS -->
+    <!-- Wheel Radius: 0.04 = 8cm diameter wheel. Change to match your actual wheel size. -->
+    <!-- Wheel Width: 0.015 = 1.5cm thickness. Adjust for wide/narrow wheels. -->
+    <!-- Wheel Mass: 0.1 = 100 grams per wheel. Heavier wheels = better traction, slower response. -->
+    <!-- Wheel Inertia: Automatically calculated from radius and mass (I = (1/12)*m*(3*r^2 + h^2)) -->
+    <!-- Macro to create wheel link with simple cylinder geometry -->
+    <xacro:macro name="wheel_link" params="name mass">
+        <link name="${ns}/${name}">
+            <inertial>
+                <mass value="${mass}"/>
+                <!-- WHEEL INERTIA CALCULATION: For 0.04m radius, 0.015m width, 0.1kg mass = 0.000067 -->
+                <!-- Adjust these values if you change wheel radius/mass substantially -->
+                <origin xyz="0 0 0" rpy="0 0 0"/>
+                <inertia ixx="0.000067" ixy="0" ixz="0" iyy="0.000067" iyz="0" izz="0.000032"/>
+            </inertial>
+            <xacro:if value="${show_helper_wheels}">
+                <visual>
+                    <geometry>
+                        <!-- WHEEL RADIUS: Change 0.04 to your wheel radius in meters -->
+                        <!-- WHEEL WIDTH: Change 0.015 to your wheel width/thickness in meters -->
+                        <cylinder radius="0.04" length="0.015"/>
+                    </geometry>
+                    <origin xyz="0 0 0" rpy="1.5707 0 0"/>
+                    <material name="Black"/>
+                </visual>
+            </xacro:if>
+            <collision>
+                <geometry>
+                    <!-- WHEEL RADIUS: Must match visual radius above -->
+                    <!-- WHEEL WIDTH: Must match visual width above -->
+                    <cylinder radius="0.04" length="0.015"/>
+                </geometry>
+                <origin xyz="0 0 0" rpy="1.5707 0 0"/>
+            </collision>
+        </link>
+    </xacro:macro>
+    <!-- Macro to create wheel joint with continuous rotation for differential drive -->
+    <xacro:macro name="wheel_joint" params="name parent child x_pos y_pos">
+        <joint name="${ns}/${name}" type="continuous">
+            <parent link="${ns}/${parent}"/>
+            <child link="${ns}/${child}"/>
+            <!-- WHEEL POSITION CONFIGURATION:
+                 - x_pos: Forward/backward from base_link center (0.05 = 5cm forward)
+                 - y_pos: Left/right position. Positive = right, negative = left
+                 - Z position: Automatically set to -0.036 (wheel radius 0.04m - 0.004m clearance)
+                 EDIT x_pos AND y_pos VALUES TO ADJUST WHEEL PLACEMENT -->
+            <origin xyz="${x_pos} ${y_pos} -0.036" rpy="0 0 0"/>
+            <!-- Rotation axis: 0 1 0 = Y-axis rotation (wheels spin side-to-side) -->
+            <axis xyz="0 1 0"/>
+            <!-- MOTOR TORQUE LIMIT (effort): 10 N⋅m default. Increase for more power, decrease for less. -->
+            <!-- MOTOR SPEED LIMIT (velocity): 2 rad/s default. Increase for faster rotation. -->
+            <limit effort="10" velocity="2"/>
+            <dynamics damping="0.1" friction="0.0"/>
+        </joint>
+    </xacro:macro>
+    <xacro:common_link name="base_link" material="Green" path="X3plus">
         <inertial>
             <origin xyz="-0.0304416859098744 4.23384368655101E-05 0.0448234503408059" rpy="0 0 0"/>
@@ -69,8 +142,41 @@
                     izz="0.0129535610833954"/>
         </inertial>
-    </common_link>
-    <fixed_joint name="base_joint" parent="base_footprint" child="base_link" xyz="0.0 0.0 0.076" rpy="0 0 0"/>
-    <fixed_joint name="base_imu" parent="base_link" child="imu_link" xyz="0.001 0.017 0.0322" rpy="0 3.1415 1.5707"/>
-    <common_link name="laser_link" material="White" path="sensor">
+    </xacro:common_link>
+    <xacro:fixed_joint name="base_joint" parent="base_footprint" child="base_link" xyz="0.0 0.0 0.076" rpy="0 0 0"/>
+    <xacro:fixed_joint name="base_imu" parent="base_link" child="imu_link" xyz="0.001 0.017 0.0322" rpy="0 3.1415 1.5707"/>
+    <!-- ==================== DIFFERENTIAL DRIVE WHEELS ==================== -->
+    <!-- CONFIGURABLE: Wheel Mass (kg). Default 0.1 = 100 grams each wheel -->
+    <!-- Change for heavier/lighter wheels. More mass = better traction but slower acceleration -->
+    <xacro:wheel_link name="left_wheel" mass="0.1"/>
+    <xacro:wheel_link name="right_wheel" mass="0.1"/>
+    <!-- CONFIGURABLE: Wheel Positions (forward/backward from base center) -->
+    <!-- Left wheel: x_pos=0.05 (5cm forward), y_pos=0.08 (8cm to the left) -->
+    <!-- Right wheel: x_pos=0.05 (5cm forward), y_pos=-0.08 (8cm to the right) -->
+    <!-- ADJUST x_pos TO MOVE WHEELS FORWARD/BACKWARD -->
+    <!-- ADJUST y_pos TO CHANGE DISTANCE BETWEEN WHEELS (wheel_separation) -->
+    <xacro:wheel_joint name="left_wheel_joint" parent="base_link" child="left_wheel" x_pos="0.05" y_pos="0.08"/>
+    <xacro:wheel_joint name="right_wheel_joint" parent="base_link" child="right_wheel" x_pos="0.05" y_pos="-0.08"/>
+    <!-- GAZEBO FRICTION PROPERTIES FOR WHEELS -->
+    <!-- mu1, mu2: Friction coefficients (0.0-1.0+). Higher = more grip. 0.8 is typical rubber on floor -->
+    <!-- kp, kd: Contact stiffness and damping. Higher kp = stiffer contact, better for rigid wheels -->
+    <gazebo reference="left_wheel">
+        <material>Gazebo/Black</material>
+        <!-- FRICTION: mu1 and mu2 control grip. 0.8 is good for rubber wheels on normal floor -->
+        <mu1>0.8</mu1>
+        <mu2>0.8</mu2>
+        <!-- CONTACT STIFFNESS: kp controls how rigid the wheel contact is -->
+        <kp>1000000.0</kp>
+        <kd>1.0</kd>
+    </gazebo>
+    <gazebo reference="right_wheel">
+        <material>Gazebo/Black</material>
+        <!-- FRICTION: mu1 and mu2 control grip. 0.8 is good for rubber wheels on normal floor -->
+        <mu1>0.8</mu1>
+        <mu2>0.8</mu2>
+        <!-- CONTACT STIFFNESS: kp controls how rigid the wheel contact is -->
+        <kp>1000000.0</kp>
+        <kd>1.0</kd>
+    </gazebo>
+    <xacro:common_link name="laser_link" material="White" path="sensor_X3plus">
         <inertial>
             <origin xyz="-0.0176558922685589 0.000671805271544437 0.0219302095894866" rpy="0 0 0"/>
@@ -79,7 +185,7 @@
                      iyy="3.89262522903605E-05" iyz="3.24809725932687E-07" izz="4.86230801106223E-05"/>
         </inertial>
-    </common_link>
-    <fixed_joint name="laser_joint" parent="base_link" child="laser_link" xyz="0.10478 0 0.0471" rpy="0 0 0"/>
-    <common_link name="camera_link" material="White" path="sensor">
+    </xacro:common_link>
+    <xacro:fixed_joint name="laser_joint" parent="base_link" child="laser_link" xyz="0.10478 0 0.0471" rpy="0 0 0"/>
+    <xacro:common_link name="camera_link" material="White" path="sensor_X3plus">
         <inertial>
             <origin xyz="0 0 0" rpy="0 0 0"/>
@@ -87,7 +193,7 @@
             <inertia ixx="0" ixy="0" ixz="0" iyy="0" iyz="0" izz="0"/>
         </inertial>
-    </common_link>
-    <fixed_joint name="camera_joint" parent="base_link" child="camera_link" xyz="-0.043645 0 0.41955" rpy="0 0 0"/>
-    <common_link name="arm_link1" material="White" path="X3plus">
+    </xacro:common_link>
+    <xacro:fixed_joint name="camera_joint" parent="base_link" child="camera_link" xyz="-0.043645 0 0.41955" rpy="0 0 0"/>
+    <xacro:common_link name="arm_link1" material="White" path="X3plus">
         <inertial>
             <origin xyz="1.99179507982521E-05 -5.98354652829568E-05 0.0114289358828097" rpy="0 0 0"/>
@@ -101,8 +207,8 @@
                     izz="1.49639510661413E-05"/>
         </inertial>
-    </common_link>
-    <revolute_joint name="arm_joint1" parent="base_link" child="arm_link1" xyz="0.09825 0 0.102" rpy="0 0 0" axisZ="-1"
+    </xacro:common_link>
+    <xacro:revolute_joint name="arm_joint1" parent="base_link" child="arm_link1" xyz="0.09825 0 0.102" rpy="0 0 0" axisZ="-1"
                     lower="-${pi/2}" upper="${pi/2}"/>
-    <common_link name="arm_link2" material="Green" path="X3plus">
+    <xacro:common_link name="arm_link2" material="Green" path="X3plus">
         <inertial>
             <origin xyz="0.024903 -0.0022632 -0.00066663" rpy="0 0 0"/>
@@ -116,8 +222,8 @@
                     izz="2.4695E-05"/>
         </inertial>
-    </common_link>
-    <revolute_joint name="arm_joint2" parent="arm_link1" child="arm_link2" xyz="0 0 0.0405"
+    </xacro:common_link>
+    <xacro:revolute_joint name="arm_joint2" parent="arm_link1" child="arm_link2" xyz="0 0 0.0405"
                     rpy="-${pi/2} 0 0" axisZ="-1" lower="-${pi/2}" upper="${pi/2}"/>
-    <common_link name="arm_link3" material="White" path="X3plus">
+    <xacro:common_link name="arm_link3" material="White" path="X3plus">
         <inertial>
             <origin xyz="0.024903 -0.0022634 -0.0013962" rpy="0 0 0"/>
@@ -131,8 +237,8 @@
                     izz="2.4695E-05"/>
         </inertial>
-    </common_link>
-    <revolute_joint name="arm_joint3" parent="arm_link2" child="arm_link3" xyz="0 -0.0829 0" rpy="0 0 0"
+    </xacro:common_link>
+    <xacro:revolute_joint name="arm_joint3" parent="arm_link2" child="arm_link3" xyz="0 -0.0829 0" rpy="0 0 0"
                     axisZ="-1" lower="-${pi/2}" upper="${pi/2}"/>
-    <common_link name="arm_link4" material="Green" path="X3plus">
+    <xacro:common_link name="arm_link4" material="Green" path="X3plus">
         <inertial>
             <origin xyz="0.036246 0.0023413 -0.0019655" rpy="0 0 0"/>
@@ -146,8 +252,8 @@
                     izz="4.1769E-05"/>
         </inertial>
-    </common_link>
-    <revolute_joint name="arm_joint4" parent="arm_link3" child="arm_link4" xyz="0 -0.0829 0" rpy="0 0 0"
+    </xacro:common_link>
+    <xacro:revolute_joint name="arm_joint4" parent="arm_link3" child="arm_link4" xyz="0 -0.0829 0" rpy="0 0 0"
                     axisZ="-1" lower="-${pi/2}" upper="${pi/2}"/>
-    <common_link name="arm_link5" material="White" path="X3plus">
+    <xacro:common_link name="arm_link5" material="White" path="X3plus">
         <inertial>
             <origin xyz="0.0023228 0.018169 0.028684" rpy="0 0 0"/>
@@ -161,8 +267,8 @@
                     izz="1.3298E-05"/>
         </inertial>
-    </common_link>
-    <revolute_joint name="arm_joint5" parent="arm_link4" child="arm_link5" xyz="-0.00215 -0.17455 0"
+    </xacro:common_link>
+    <xacro:revolute_joint name="arm_joint5" parent="arm_link4" child="arm_link5" xyz="-0.00215 -0.17455 0"
                     rpy="${pi/2} 0 0" axisZ="1" lower="-${pi/2}" upper="${pi}"/>
-    <common_link name="rlink1" material="Green" path="X3plus">
+    <xacro:common_link name="rlink1" material="Green" path="X3plus">
         <inertial>
             <origin xyz="0.00653227489887718 0.000416767821288678 0.000980984132845697" rpy="0 0 0"/>
@@ -176,8 +282,8 @@
                     izz="1.99277285249309E-07"/>
         </inertial>
-    </common_link>
-    <revolute_joint name="grip_joint" parent="arm_link5" child="rlink1" xyz="-0.0035 -0.012625 -0.0685"
+    </xacro:common_link>
+    <xacro:revolute_joint name="grip_joint" parent="arm_link5" child="rlink1" xyz="-0.0035 -0.012625 -0.0685"
                     rpy="0 -${pi/2} 0" axisZ="1" lower="-${pi/2}" upper="0"/>
-    <common_link name="rlink2" material="Green" path="X3plus">
+    <xacro:common_link name="rlink2" material="Green" path="X3plus">
         <inertial>
             <origin xyz="0.021158 0.0063295 -0.0030251" rpy="0 0 0"/>
@@ -191,7 +297,7 @@
                     izz="6.6364E-07"/>
         </inertial>
-    </common_link>
-    <continuous_joint name="rlink_joint2" parent="rlink1" child="rlink2" xyz="0.03 -0.00075429 0" rpy="0 0 0" mimic="-1"/>
-    <common_link name="rlink3" material="Green" path="X3plus">
+    </xacro:common_link>
+    <xacro:continuous_joint name="rlink_joint2" parent="rlink1" child="rlink2" xyz="0.03 -0.00075429 0" rpy="0 0 0" mimic="-1"/>
+    <xacro:common_link name="rlink3" material="Green" path="X3plus">
         <inertial>
             <origin xyz="0.014355 1.1499E-05 -0.0033992" rpy="0 0 0"/>
@@ -205,8 +311,8 @@
                     izz="1.3089E-07"/>
         </inertial>
-    </common_link>
-    <continuous_joint name="rlink_joint3" parent="arm_link5" child="rlink3" xyz="-0.0035 -0.0045 -0.0505"
+    </xacro:common_link>
+    <xacro:continuous_joint name="rlink_joint3" parent="arm_link5" child="rlink3" xyz="-0.0035 -0.0045 -0.0505"
                       rpy="0 -${pi/2} 0" mimic="1"/>
-    <common_link name="llink1" material="Green" path="X3plus">
+    <xacro:common_link name="llink1" material="Green" path="X3plus">
         <inertial>
             <origin xyz="0.00628617364795481 -0.000318530407893543 0.00100000338924466" rpy="0 0 0"/>
@@ -220,8 +326,8 @@
                     izz="2.00283878176223E-07"/>
         </inertial>
-    </common_link>
-    <continuous_joint name="llink_joint1" parent="arm_link5" child="llink1" xyz="-0.0035 0.012375 -0.0685"
+    </xacro:common_link>
+    <xacro:continuous_joint name="llink_joint1" parent="arm_link5" child="llink1" xyz="-0.0035 0.012375 -0.0685"
                       rpy="0 -${pi/2} 0" mimic="-1"/>
-    <common_link name="llink2" material="Green" path="X3plus">
+    <xacro:common_link name="llink2" material="Green" path="X3plus">
         <inertial>
             <origin xyz="0.021159 -0.0063248 -0.0030251" rpy="0 0 0"/>
@@ -230,8 +336,8 @@
                      izz="6.6364E-07"/>
         </inertial>
-    </common_link>
-    <continuous_joint name="llink_joint2" parent="llink1" child="llink2" xyz="0.03 0.00065104 0" rpy="0 0 0"
+    </xacro:common_link>
+    <xacro:continuous_joint name="llink_joint2" parent="llink1" child="llink2" xyz="0.03 0.00065104 0" rpy="0 0 0"
                       mimic="1"/>
-    <common_link name="llink3" material="Green" path="X3plus">
+    <xacro:common_link name="llink3" material="Green" path="X3plus">
         <inertial>
             <origin xyz="0.014354 -7.4795E-05 -0.0033992" rpy="0 0 0"/>
@@ -240,8 +346,8 @@
                      izz="1.3089E-07"/>
         </inertial>
-    </common_link>
-    <continuous_joint name="llink_joint3" parent="arm_link5" child="llink3" xyz="-0.0035 0.0045 -0.0505"
+    </xacro:common_link>
+    <xacro:continuous_joint name="llink_joint3" parent="arm_link5" child="llink3" xyz="-0.0035 0.0045 -0.0505"
                       rpy="0 -${pi/2} 0" mimic="-1"/>
-    <common_link name="mono_link" material="White" path="sensor">
+    <xacro:common_link name="mono_link" material="White" path="sensor_X3plus">
         <inertial>
             <origin xyz="5.8458E-05 0.0095015 -0.0014824" rpy="0 0 0"/>
@@ -250,6 +356,66 @@
                      izz="2.5696E-06"/>
         </inertial>
-    </common_link>
-    <fixed_joint name="mono_joint" parent="arm_link4" child="mono_link" xyz="-0.0481 -0.05145 -0.0022"
+    </xacro:common_link>
+    <xacro:fixed_joint name="mono_joint" parent="arm_link4" child="mono_link" xyz="0.0481 -0.05145 -0.0022"
                  rpy="${pi/2} 0 0"/>
+    <!-- ==================== ARM INITIAL POSITIONS FOR GAZEBO ==================== -->
+    <!-- Set default joint positions to match RViz (all at 0 radians) -->
+    <gazebo reference="arm_joint1">
+        <implicitSpringDamper>true</implicitSpringDamper>
+        <initial_position>0</initial_position>
+    </gazebo>
+    <gazebo reference="arm_joint2">
+        <implicitSpringDamper>true</implicitSpringDamper>
+        <initial_position>0</initial_position>
+    </gazebo>
+    <gazebo reference="arm_joint3">
+        <implicitSpringDamper>true</implicitSpringDamper>
+        <initial_position>0</initial_position>
+    </gazebo>
+    <gazebo reference="arm_joint4">
+        <implicitSpringDamper>true</implicitSpringDamper>
+        <initial_position>0</initial_position>
+    </gazebo>
+    <gazebo reference="arm_joint5">
+        <implicitSpringDamper>true</implicitSpringDamper>
+        <initial_position>0</initial_position>
+    </gazebo>
+    <!-- ==================== GAZEBO DIFFERENTIAL DRIVE PLUGIN ==================== -->
+    <!-- This plugin controls the wheels for differential drive (tank-style) movement -->
+    <!-- CONFIGURABLE PARAMETERS BELOW: -->
+    <!-- NOTE: Plugin must be linked to base_link for proper operation -->
+    <gazebo reference="base_link">
+        <plugin name="diff_drive" filename="libgazebo_ros_diff_drive.so">
+            <!-- Joint names: Must match the joint names defined in the URDF above -->
+            <!-- NOTE: No namespace prefix - joints are named without x3plus/ prefix -->
+            <left_joint>left_wheel_joint</left_joint>
+            <right_joint>right_wheel_joint</right_joint>
+            <!-- WHEEL SEPARATION: Distance between left and right wheels in meters -->
+            <!-- Default: 0.16 (16cm). This should match Y positions: abs(0.08 - (-0.08)) = 0.16 -->
+            <!-- IMPORTANT: Must be consistent with your wheel y_pos values! -->
+            <wheel_separation>0.16</wheel_separation>
+            <!-- WHEEL DIAMETER: Diameter of wheels (2 * radius) -->
+            <!-- Default: 0.08 (8cm) matches radius 0.04m. Change if you modified wheel radius -->
+            <wheel_diameter>0.08</wheel_diameter>
+            <!-- MOTOR TORQUE: Maximum torque output (N⋅m). Default 10. -->
+            <!-- Increase for more powerful drive, decrease for gentler acceleration -->
+            <max_wheel_torque>10</max_wheel_torque>
+            <!-- ACCELERATION LIMIT: Maximum wheel acceleration (rad/s^2). Default 1.0 -->
+            <!-- Increase for snappier response, decrease for smoother acceleration -->
+            <max_wheel_accel>1.0</max_wheel_accel>
+            <!-- ROS TOPICS: Names of command and odometry topics -->
+            <!-- Send movement commands to: ros2 topic pub /cmd_vel geometry_msgs/Twist ... -->
+            <command_topic>cmd_vel</command_topic>
+            <odometry_topic>odom</odometry_topic>
+            <odometry_frame>odom</odometry_frame>
+            <!-- CRITICAL: Use base_footprint as the robot base frame (no namespace) -->
+            <robot_base_frame>base_footprint</robot_base_frame>
+            <!-- ODOMETRY PUBLISHING: Whether to publish position estimates -->
+            <publish_odom>true</publish_odom>
+            <!-- Publish TF transforms for odometry (usually false for real robots) -->
+            <publish_odom_tf>false</publish_odom_tf>
+            <!-- UPDATE RATE: How often to update physics (Hz). 30 is typical for simulations -->
+            <update_rate>30</update_rate>
+        </plugin>
+    </gazebo>
 </robot>
