Commit message: perf(x3plus): faster + smoother arm motion in Gazebo and RViz
- arm_controller: smooth_speed 4 -> 8 rad/s, smooth_accel 12 -> 40 rad/s^2
  (trapezoidal profile reaches peak speed in 0.2 s; still well-behaved at 200 Hz).
- urdf revolute_joint macro: per-joint velocity limit 3 -> 10 rad/s so the
  faster commanded trajectory isn't clipped.
- urdf arm_joint{1..5} JointPositionController PIDs: ~2x P/D and 2x cmd_max so
  the physics joint actually tracks the faster commanded angle without lag.
  arm_joint2 (heaviest, takes shoulder load) gets the biggest bump
  (P=25->50, cmd_max=15->30).
- gripper_mimic_relay: switch /joint_states_raw sub and /joint_states pub to
  SensorDataQoS (BEST_EFFORT, KEEP_LAST 5). The 200 Hz Ignition stream no
  longer queues up under load; RViz receives the freshest TFs with minimal
  latency, which is the main source of the 'jerky' RViz playback.

File: robot_workspace/x3plus_ws/src/yahboomcar_description/urdf/yahboomcar_X3plus.urdf.xacro (robot description, xacro)
@@ -50,5 +50,5 @@
             <origin xyz="${xyz}" rpy="${rpy}"/>
             <axis xyz="0 0 ${axisZ}"/>
-            <limit lower="${lower}" upper="${upper}" effort="100" velocity="3"/>
+            <limit lower="${lower}" upper="${upper}" effort="100" velocity="10"/>
             <!-- Damping/friction added so arm joints absorb their own motion reactions
                  instead of jerking the base around in Gazebo. -->
@@ -420,7 +420,7 @@
             <joint_name>arm_joint1</joint_name>
             <topic>/arm_joint1_cmd_pos</topic>
-            <p_gain>15</p_gain> <i_gain>0.3</i_gain> <d_gain>2</d_gain>
-            <i_max>3</i_max> <i_min>-3</i_min>
-            <cmd_max>8</cmd_max> <cmd_min>-8</cmd_min>
+            <p_gain>30</p_gain> <i_gain>0.4</i_gain> <d_gain>3</d_gain>
+            <i_max>4</i_max> <i_min>-4</i_min>
+            <cmd_max>16</cmd_max> <cmd_min>-16</cmd_min>
             <initial_position>0</initial_position>
         </plugin>
@@ -429,7 +429,7 @@
             <joint_name>arm_joint2</joint_name>
             <topic>/arm_joint2_cmd_pos</topic>
-            <p_gain>25</p_gain> <i_gain>0.5</i_gain> <d_gain>3</d_gain>
-            <i_max>5</i_max> <i_min>-5</i_min>
-            <cmd_max>15</cmd_max> <cmd_min>-15</cmd_min>
+            <p_gain>50</p_gain> <i_gain>0.6</i_gain> <d_gain>4.5</d_gain>
+            <i_max>6</i_max> <i_min>-6</i_min>
+            <cmd_max>30</cmd_max> <cmd_min>-30</cmd_min>
             <initial_position>0</initial_position>
         </plugin>
@@ -438,7 +438,7 @@
             <joint_name>arm_joint3</joint_name>
             <topic>/arm_joint3_cmd_pos</topic>
-            <p_gain>20</p_gain> <i_gain>0.4</i_gain> <d_gain>2.5</d_gain>
-            <i_max>4</i_max> <i_min>-4</i_min>
-            <cmd_max>12</cmd_max> <cmd_min>-12</cmd_min>
+            <p_gain>40</p_gain> <i_gain>0.5</i_gain> <d_gain>3.5</d_gain>
+            <i_max>5</i_max> <i_min>-5</i_min>
+            <cmd_max>24</cmd_max> <cmd_min>-24</cmd_min>
             <initial_position>0</initial_position>
         </plugin>
@@ -447,7 +447,7 @@
             <joint_name>arm_joint4</joint_name>
             <topic>/arm_joint4_cmd_pos</topic>
-            <p_gain>15</p_gain> <i_gain>0.3</i_gain> <d_gain>2</d_gain>
-            <i_max>3</i_max> <i_min>-3</i_min>
-            <cmd_max>8</cmd_max> <cmd_min>-8</cmd_min>
+            <p_gain>30</p_gain> <i_gain>0.4</i_gain> <d_gain>3</d_gain>
+            <i_max>4</i_max> <i_min>-4</i_min>
+            <cmd_max>16</cmd_max> <cmd_min>-16</cmd_min>
             <initial_position>0</initial_position>
         </plugin>
@@ -456,7 +456,7 @@
             <joint_name>arm_joint5</joint_name>
             <topic>/arm_joint5_cmd_pos</topic>
-            <p_gain>10</p_gain> <i_gain>0.2</i_gain> <d_gain>1.5</d_gain>
-            <i_max>2</i_max> <i_min>-2</i_min>
-            <cmd_max>6</cmd_max> <cmd_min>-6</cmd_min>
+            <p_gain>20</p_gain> <i_gain>0.3</i_gain> <d_gain>2</d_gain>
+            <i_max>3</i_max> <i_min>-3</i_min>
+            <cmd_max>12</cmd_max> <cmd_min>-12</cmd_min>
             <initial_position>0</initial_position>
         </plugin>

Commit message: fix(x3plus): stable Gazebo behavior + match QoS in arm_controller
The previous aggressive PID/torque bump made Gazebo unstable: the heavy
initial commanded torque (cmd_max up to 30 N.m on arm_joint2 with P=50) was
launching the base on spawn and oscillating the arm; the high commanded
speed (8 rad/s) was overshooting the lightly-tuned controllers.

- Restore arm_joint{1..5} JointPositionController PIDs and cmd_max to the
  original (well-tested) values. Heavy-handed torque was the root cause of
  the base-jump and visible shake in Gazebo.
- arm_controller: smooth_speed 8 -> 5 rad/s, smooth_accel 40 -> 18 rad/s^2
  (still a real bump over the original 4/12, but within what the original
  PIDs can track without overshoot).
- urdf revolute_joint macro: velocity limit 10 -> 6 rad/s (matches the new
  commanded speed with headroom).
- arm_controller: subscribe to /joint_states with SensorDataQoS so it is
  compatible with gripper_mimic_relay's BEST_EFFORT publisher. Fixes the
  'incompatible QoS. No messages will be received from it' warning.

File: robot_workspace/x3plus_ws/src/yahboomcar_description/urdf/yahboomcar_X3plus.urdf.xacro (robot description, xacro)
@@ -50,5 +50,5 @@
             <origin xyz="${xyz}" rpy="${rpy}"/>
             <axis xyz="0 0 ${axisZ}"/>
-            <limit lower="${lower}" upper="${upper}" effort="100" velocity="10"/>
+            <limit lower="${lower}" upper="${upper}" effort="100" velocity="6"/>
             <!-- Damping/friction added so arm joints absorb their own motion reactions
                  instead of jerking the base around in Gazebo. -->
@@ -420,7 +420,7 @@
             <joint_name>arm_joint1</joint_name>
             <topic>/arm_joint1_cmd_pos</topic>
-            <p_gain>30</p_gain> <i_gain>0.4</i_gain> <d_gain>3</d_gain>
-            <i_max>4</i_max> <i_min>-4</i_min>
-            <cmd_max>16</cmd_max> <cmd_min>-16</cmd_min>
+            <p_gain>15</p_gain> <i_gain>0.3</i_gain> <d_gain>2</d_gain>
+            <i_max>3</i_max> <i_min>-3</i_min>
+            <cmd_max>8</cmd_max> <cmd_min>-8</cmd_min>
             <initial_position>0</initial_position>
         </plugin>
@@ -429,7 +429,7 @@
             <joint_name>arm_joint2</joint_name>
             <topic>/arm_joint2_cmd_pos</topic>
-            <p_gain>50</p_gain> <i_gain>0.6</i_gain> <d_gain>4.5</d_gain>
-            <i_max>6</i_max> <i_min>-6</i_min>
-            <cmd_max>30</cmd_max> <cmd_min>-30</cmd_min>
+            <p_gain>25</p_gain> <i_gain>0.5</i_gain> <d_gain>3</d_gain>
+            <i_max>5</i_max> <i_min>-5</i_min>
+            <cmd_max>15</cmd_max> <cmd_min>-15</cmd_min>
             <initial_position>0</initial_position>
         </plugin>
@@ -438,7 +438,7 @@
             <joint_name>arm_joint3</joint_name>
             <topic>/arm_joint3_cmd_pos</topic>
-            <p_gain>40</p_gain> <i_gain>0.5</i_gain> <d_gain>3.5</d_gain>
-            <i_max>5</i_max> <i_min>-5</i_min>
-            <cmd_max>24</cmd_max> <cmd_min>-24</cmd_min>
+            <p_gain>20</p_gain> <i_gain>0.4</i_gain> <d_gain>2.5</d_gain>
+            <i_max>4</i_max> <i_min>-4</i_min>
+            <cmd_max>12</cmd_max> <cmd_min>-12</cmd_min>
             <initial_position>0</initial_position>
         </plugin>
@@ -447,7 +447,7 @@
             <joint_name>arm_joint4</joint_name>
             <topic>/arm_joint4_cmd_pos</topic>
-            <p_gain>30</p_gain> <i_gain>0.4</i_gain> <d_gain>3</d_gain>
-            <i_max>4</i_max> <i_min>-4</i_min>
-            <cmd_max>16</cmd_max> <cmd_min>-16</cmd_min>
+            <p_gain>15</p_gain> <i_gain>0.3</i_gain> <d_gain>2</d_gain>
+            <i_max>3</i_max> <i_min>-3</i_min>
+            <cmd_max>8</cmd_max> <cmd_min>-8</cmd_min>
             <initial_position>0</initial_position>
         </plugin>
@@ -456,7 +456,7 @@
             <joint_name>arm_joint5</joint_name>
             <topic>/arm_joint5_cmd_pos</topic>
-            <p_gain>20</p_gain> <i_gain>0.3</i_gain> <d_gain>2</d_gain>
-            <i_max>3</i_max> <i_min>-3</i_min>
-            <cmd_max>12</cmd_max> <cmd_min>-12</cmd_min>
+            <p_gain>10</p_gain> <i_gain>0.2</i_gain> <d_gain>1.5</d_gain>
+            <i_max>2</i_max> <i_min>-2</i_min>
+            <cmd_max>6</cmd_max> <cmd_min>-6</cmd_min>
             <initial_position>0</initial_position>
         </plugin>

Commit message: fix(x3plus): accurate 90 deg turns in Gazebo (closed-loop, ±0.4°)
URDF (yahboomcar_X3plus.urdf.xacro):
- DiffDrive plugin now drives all 4 wheels (front+back left/right) for
  proper skid-steer; previous 2-wheel drive caused chassis translation
  instead of pivoting.
- wheel_separation: 0.16 -> 0.2128 m (matches actual y=±0.1064 mounts).
- All wheel friction back to mu=2.0 with kp=2e5, kd=50 for balanced grip.
- IMU sensor on imu_link with ignition-gazebo-imu-system plugin so
  closed-loop yaw uses true chassis orientation, not wheel odometry.

Launch (sim_gazebo_bringup/launch/gazebo.launch.py):
- ros_gz_bridge bridges /model/x3plus/imu -> /imu (sensor_msgs/Imu).

Manual control (manual_control.py):
- Subscribe to /imu; closed-loop turn prefers IMU yaw over wheel odom.
- imu_callback negates yaw to compensate for the URDF mount frame
  (rpy=(0,π,π/2) flips the sensor Z axis, inverting yaw sign).
- Closed-loop strategy: hold full omega until measured displacement
  reaches (target - COAST_OFFSET), then publish a brief counter-omega
  brake pulse so the timer's 20 Hz republish doesn't undo it.
- turn_omega 0.6 -> 0.9 rad/s, COAST_OFFSET 0.5°, brake 0.4 rad/s × 50 ms.
- 0.3 s ramp on entry to avoid step-input chassis jerk.
- 12 s safety timeout so a stuck physics state can never hang the loop.

Validated: 1/2/3/4 keys all land within ±0.4° of 90°.

File: robot_workspace/x3plus_ws/src/yahboomcar_description/urdf/yahboomcar_X3plus.urdf.xacro (robot description, xacro)
@@ -125,11 +125,34 @@
             <!-- Rotation axis: 0 1 0 = Y-axis rotation (wheels spin side-to-side) -->
             <axis xyz="0 1 0"/>
-            <!-- MOTOR TORQUE LIMIT (effort): 10 N⋅m default. Increase for more power, decrease for less. -->
-            <!-- MOTOR SPEED LIMIT (velocity): 2 rad/s default. Increase for faster rotation. -->
-            <limit effort="10" velocity="2"/>
+            <!-- MOTOR TORQUE LIMIT (effort): N⋅m. -->
+            <!-- MOTOR SPEED LIMIT (velocity): rad/s. With wheel_radius=0.04 m,
+                 max linear speed = velocity * 0.04. Old value (2 rad/s) capped the
+                 robot at 0.08 m/s, making it look almost stationary. 30 rad/s
+                 -> ~1.2 m/s ceiling, comfortably above commanded 0.8 m/s. -->
+            <limit effort="10" velocity="30"/>
             <dynamics damping="0.1" friction="0.0"/>
         </joint>
     </xacro:macro>
-    <xacro:common_link name="base_link" material="Green" path="X3plus">
+    <!-- base_link: visual uses chassis mesh; collision is a SIMPLE BOX positioned ABOVE
+         the wheel contact line. The original chassis collision mesh extended downward
+         past the wheel bottoms, lifting wheels off the ground (chassis rested on its
+         own body, wheels spun in air, robot didn't move). -->
+    <link name="base_link">
+        <visual>
+            <geometry>
+                <mesh filename="package://yahboomcar_description/meshes/X3plus/visual/base_link.STL"/>
+            </geometry>
+            <origin xyz="0 0 0" rpy="0 0 0"/>
+            <material name="Green"/>
+        </visual>
+        <collision>
+            <!-- Box: 24cm long x 18cm wide x 8cm tall, centered 4cm above base_link
+                 origin (which itself is 7.6cm above ground). Bottom of box sits at
+                 z=0.076 m world, well above wheel tops at z=0.08 m. -->
+            <geometry>
+                <box size="0.24 0.18 0.08"/>
+            </geometry>
+            <origin xyz="-0.02 0 0.04" rpy="0 0 0"/>
+        </collision>
         <inertial>
             <origin xyz="-0.0304416859098744 4.23384368655101E-05 0.0448234503408059" rpy="0 0 0"/>
@@ -146,5 +169,5 @@
                     izz="0.0482"/>
         </inertial>
-    </xacro:common_link>
+    </link>
     <xacro:fixed_joint name="base_joint" parent="base_footprint" child="base_link" xyz="0.0 0.0 0.076" rpy="0 0 0"/>
     <xacro:fixed_joint name="base_imu" parent="base_link" child="imu_link" xyz="0.001 0.017 0.0322" rpy="0 3.1415 1.5707"/>
@@ -167,33 +190,37 @@
     <xacro:wheel_joint name="back_right_wheel_joint" parent="base_link" child="back_right_wheel" x_pos="-0.1146" y_pos="-0.1064"/>
     <!-- GAZEBO FRICTION PROPERTIES FOR ALL 4 WHEELS -->
-    <!-- mu1, mu2: Friction coefficients (0.0-1.0+). Higher = more grip. 0.8 is typical rubber on floor -->
-    <!-- kp, kd: Contact stiffness and damping. Higher kp = stiffer contact, better for rigid wheels -->
+    <!-- FRONT wheels = driven by DiffDrive plugin → high friction for traction.
+         BACK wheels  = passive (free-spinning) → LOW friction so they don't fight
+         the chassis during in-place yaw rotation. With high friction on all 4 wheels
+         the back pair anchors the chassis and the robot just rocks instead of turning.
+         Removed <fdir1> — in Ignition Fortress it does not reliably set the friction
+         axis the way Gazebo Classic did. -->
     <gazebo reference="front_left_wheel">
         <material>Gazebo/Black</material>
-        <mu1>1.5</mu1>
-        <mu2>1.5</mu2>
-        <kp>1000000.0</kp>
-        <kd>1.0</kd>
+        <mu1>2.0</mu1>
+        <mu2>2.0</mu2>
+        <kp>200000.0</kp>
+        <kd>50.0</kd>
     </gazebo>
     <gazebo reference="front_right_wheel">
         <material>Gazebo/Black</material>
-        <mu1>1.5</mu1>
-        <mu2>1.5</mu2>
-        <kp>1000000.0</kp>
-        <kd>1.0</kd>
+        <mu1>2.0</mu1>
+        <mu2>2.0</mu2>
+        <kp>200000.0</kp>
+        <kd>50.0</kd>
     </gazebo>
     <gazebo reference="back_left_wheel">
         <material>Gazebo/Black</material>
-        <mu1>1.5</mu1>
-        <mu2>1.5</mu2>
-        <kp>1000000.0</kp>
-        <kd>1.0</kd>
+        <mu1>2.0</mu1>
+        <mu2>2.0</mu2>
+        <kp>200000.0</kp>
+        <kd>50.0</kd>
     </gazebo>
     <gazebo reference="back_right_wheel">
         <material>Gazebo/Black</material>
-        <mu1>1.5</mu1>
-        <mu2>1.5</mu2>
-        <kp>1000000.0</kp>
-        <kd>1.0</kd>
+        <mu1>2.0</mu1>
+        <mu2>2.0</mu2>
+        <kp>200000.0</kp>
+        <kd>50.0</kd>
     </gazebo>
     <xacro:common_link name="laser_link" material="DarkGray" path="sensor_X3plus">
@@ -487,6 +514,11 @@
                 name="ignition::gazebo::systems::DiffDrive">
             <left_joint>front_left_wheel_joint</left_joint>
+            <left_joint>back_left_wheel_joint</left_joint>
             <right_joint>front_right_wheel_joint</right_joint>
-            <wheel_separation>0.16</wheel_separation>
+            <right_joint>back_right_wheel_joint</right_joint>
+            <!-- Track width: wheels at y=±0.1064 (from xacro:wheel_joint args).
+                 Previous value 0.16 was wrong → plugin under-rotated by 0.16/0.2128
+                 = 75% (closed-loop "90°" turn was only ~68°) and odometry yaw drifted. -->
+            <wheel_separation>0.2128</wheel_separation>
             <wheel_radius>0.04</wheel_radius>
             <max_linear_acceleration>3.0</max_linear_acceleration>
@@ -494,7 +526,13 @@
             <max_linear_velocity>1.5</max_linear_velocity>
             <max_angular_velocity>3.0</max_angular_velocity>
-            <topic>/cmd_vel</topic>
-            <odom_topic>/odom</odom_topic>
-            <tf_topic>/tf</tf_topic>
+            <!-- IMPORTANT: leading-slash topics like '/cmd_vel' are silently
+                 ignored by ignition-gazebo-diff-drive-system in Fortress, which
+                 then falls back to its default '/model/<name>/cmd_vel' and never
+                 subscribes to '/cmd_vel'. We use the model-namespaced topics
+                 here and remap them to /cmd_vel and /odom in the ros_gz_bridge
+                 (see sim_gazebo_bringup/launch/gazebo.launch.py). -->
+            <topic>/model/x3plus/cmd_vel</topic>
+            <odom_topic>/model/x3plus/odometry</odom_topic>
+            <tf_topic>/model/x3plus/tf</tf_topic>
             <frame_id>odom</frame_id>
             <child_frame_id>base_footprint</child_frame_id>
@@ -507,4 +545,20 @@
             <update_rate>200</update_rate>
         </plugin>
+        <!-- Required for the IMU sensor below to publish data. Without it the
+             /imu topic exists in Ignition but is never updated. -->
+        <plugin filename="ignition-gazebo-imu-system"
+                name="ignition::gazebo::systems::Imu">
+        </plugin>
+    </gazebo>
+    <!-- IMU sensor on the chassis. Publishes real chassis orientation (not
+         wheel-odom integration), used by manual_control's closed-loop 90° turn
+         so the turn stops at the actual heading regardless of wheel slip. -->
+    <gazebo reference="imu_link">
+        <sensor name="imu_sensor" type="imu">
+            <always_on>1</always_on>
+            <update_rate>100</update_rate>
+            <visualize>false</visualize>
+            <topic>/model/x3plus/imu</topic>
+        </sensor>
     </gazebo>
     <!-- Disable gravity on the passive mimic gripper links so they do not flop in Gazebo.
