Commit message: pick-and-place: tuned pick config with 6cm standoff, 30mu friction, 20g cube, static wall, landing pad, faster gripper

File: robot_workspace/x3plus_ws/src/sim_gazebo_bringup/scripts/yahboomcar_description/urdf/yahboomcar_X3plus.urdf.xacro (robot description, xacro)
@@ -652,13 +652,16 @@
         </sensor>
     </gazebo>
-    <!-- Disable gravity on the passive mimic gripper links so they do not flop in Gazebo.
+    <!-- Enable gravity on the passive mimic gripper links so they do not flop in Gazebo.
          Mimic constraints are not enforced by Ignition physics, but with gravity off
-         these links remain at their spawn pose instead of falling free.                  -->
-    <gazebo reference="llink1"><gravity>0</gravity><collision><surface><contact><collide_bitmask>0x00</collide_bitmask></contact></surface></collision></gazebo>
-    <gazebo reference="llink2"><gravity>0</gravity><collision><surface><contact><collide_bitmask>0x00</collide_bitmask></contact></surface></collision></gazebo>
-    <gazebo reference="llink3"><gravity>0</gravity><collision><surface><contact><collide_bitmask>0x00</collide_bitmask></contact></surface></collision></gazebo>
-    <gazebo reference="rlink1"><gravity>0</gravity><collision><surface><contact><collide_bitmask>0x00</collide_bitmask></contact></surface></collision></gazebo>
-    <gazebo reference="rlink2"><gravity>0</gravity><collision><surface><contact><collide_bitmask>0x00</collide_bitmask></contact></surface></collision></gazebo>
-    <gazebo reference="rlink3"><gravity>0</gravity><collision><surface><contact><collide_bitmask>0x00</collide_bitmask></contact></surface></collision></gazebo>
+         these links remain at their spawn pose instead of falling free.
+         collide_bitmask=0xFF enables collision with everything so the fingers
+         can actually grip the cube.  mu1=mu2=30.0 provides high friction to
+         prevent the cube from sliding.                                       -->
+    <gazebo reference="llink1"><gravity>0</gravity><mu1>30.0</mu1><mu2>30.0</mu2><collision><surface><contact><collide_bitmask>0xFF</collide_bitmask></contact></surface></collision></gazebo>
+    <gazebo reference="llink2"><gravity>0</gravity><mu1>30.0</mu1><mu2>30.0</mu2><collision><surface><contact><collide_bitmask>0xFF</collide_bitmask></contact></surface></collision></gazebo>
+    <gazebo reference="llink3"><gravity>0</gravity><mu1>30.0</mu1><mu2>30.0</mu2><collision><surface><contact><collide_bitmask>0xFF</collide_bitmask></contact></surface></collision></gazebo>
+    <gazebo reference="rlink1"><gravity>0</gravity><mu1>30.0</mu1><mu2>30.0</mu2><collision><surface><contact><collide_bitmask>0xFF</collide_bitmask></contact></surface></collision></gazebo>
+    <gazebo reference="rlink2"><gravity>0</gravity><mu1>30.0</mu1><mu2>30.0</mu2><collision><surface><contact><collide_bitmask>0xFF</collide_bitmask></contact></surface></collision></gazebo>
+    <gazebo reference="rlink3"><gravity>0</gravity><mu1>30.0</mu1><mu2>30.0</mu2><collision><surface><contact><collide_bitmask>0xFF</collide_bitmask></contact></surface></collision></gazebo>
     <!-- ==================== LEGACY GAZEBO CLASSIC DIFF DRIVE (DISABLED) ==================== -->
     <!-- The old Gazebo Classic libgazebo_ros_diff_drive.so plugin is not loadable in

Commit message: updated vision same as manufacturer

File: robot_workspace/x3plus_ws/src/sim_gazebo_bringup/scripts/yahboomcar_description/urdf/yahboomcar_X3plus.urdf.xacro (robot description, xacro)
@@ -56,14 +56,11 @@
         </joint>
     </xacro:macro>
-    <!-- Gripper finger joint (was 'continuous_joint' macro).
-         IMPORTANT: <mimic> has been REMOVED. In Ignition Fortress the <mimic>
-         tag conflicts with the per-joint JointPositionController plugins
-         (sometimes kinematically locking the joint, sometimes letting it
-         shake) and produced asymmetric behavior between the L and R fingers.
-         The gripper_mimic_relay node now performs the mimic in software by
-         fanning out /grip_joint_cmd_pos to each /<joint>_cmd_pos with the
-         multiplier baked in, and by republishing the actual Gazebo joint
-         angles into /joint_states for RViz/RSP. The 'mimic' parameter is
-         kept for backward signature compatibility but is unused. -->
+    <!-- Gripper finger joint macro.
+         <mimic> tags are emitted so robot_state_publisher can compute finger
+         link TF positions (rlink2/llink2 etc.) from the master grip_joint.
+         Ignition Fortress ignores <mimic> for physics — actual finger motion
+         is driven by per-joint JointPositionController plugins fed by
+         gripper_mimic_relay. The relay also strips mimic joints from
+         /joint_states_raw so RSP recomputes them from the URDF <mimic>. -->
     <xacro:macro name="continuous_joint" params="name parent child xyz rpy mimic">
         <joint name="${ns}/${name}" type="revolute">
@@ -79,4 +76,10 @@
                  while only rlink_joint2 (under load asymmetry) overshot. -->
             <dynamics damping="0.05" friction="0.005"/>
+            <!-- <mimic> tag: required by robot_state_publisher to compute finger
+                 link TF positions from the master grip_joint. Ignition Fortress
+                 ignores <mimic> for physics (handled by JointPositionController
+                 plugins + gripper_mimic_relay), but RSP needs it to publish
+                 rlink2/llink2/rlink3/llink3 frames in the TF tree. -->
+            <mimic joint="grip_joint" multiplier="${mimic}" offset="0"/>
         </joint>
     </xacro:macro>
