Commit message: Fix 4-bar gripper: rigid assembly + fixes
- Collapse 4-bar into two rigid sub-assemblies (right/left finger) driven by single master joint + mirror
  * rlink_joint2/3, llink_joint2/3: continuous -> FIXED (pads/rockers rigid)
  * llink_joint1: continuous -> REVOLUTE driven by mirror of grip_joint via relay
  * Removed 4 PID controllers (kept only llink_joint1)
- Replace wide grey cube_platform with narrow 2cm invisible post under cube (z=0.06)
  * Wheels straddle post, no more rear-wheel collision
- Tighten grip: GRIPPER_HOLD_CUBE -0.37 -> -0.23 (pads touch cube sides)
- Fix NameError: cube_target_z -> define target_z/dz in RELEASE_WAIT
- RViz: 3 RobotModels with TF prefixes (robot_1/2/3), TF frame size 0.2m
- World: cube at z=0.06 on narrow post, sink static, no ODE bucket overflow
- Sink: static=true (cannot be displaced)
- Launch: added gui:=false use_rviz:=true support for headless+RViz

File: robot_workspace/x3plus_ws/src/sim_gazebo_bringup/scripts/yahboomcar_description/urdf/yahboomcar_X3plus.urdf.xacro (robot description, xacro)
@@ -103,10 +103,9 @@
                  tiny 1-gram finger links, so 4 of 5 mimic joints stayed frozen
                  while only rlink_joint2 (under load asymmetry) overshot. -->
-            <dynamics damping="0.05" friction="0.005"/>
+             <dynamics damping="0.05" friction="0.005"/>
             <!-- <mimic> tag: required by robot_state_publisher to compute finger
-                 link TF positions from the master grip_joint. Ignition Fortress
-                 ignores <mimic> for physics (handled by JointPositionController
-                 plugins + gripper_mimic_relay), but RSP needs it to publish
-                 rlink2/llink2 frames in the TF tree. -->
+                 link TF positions from the master grip_joint. Gazebo Sim ignores
+                 <mimic> for physics (handled by JointPositionController plugins
+                 + gripper_mimic_relay), but RSP needs it for TF. -->
             <mimic joint="grip_joint" multiplier="${mimic}" offset="0"/>
         </joint>
@@ -441,12 +440,8 @@
     <xacro:continuous_joint name="rlink_joint2" parent="rlink1" child="rlink2" xyz="0.03 -0.00075429 0" rpy="0 0 0" mimic="-1"/>
     <!-- rlink3 / rlink_joint3: RIGHT 4-bar ROCKER.
-         Parented to arm_link5 and driven by mimic=+1 so it rotates by
-         the same angle as the input crank rlink1.  Together with the
+         Parented to arm_link5 and driven by mimic=-1 so it rotates in the
+         SAME direction as the input crank rlink1.  Together with the
          rlink_joint2 mimic this forms the parallelogram four-bar that
-         keeps the pad parallel through the whole grip range.
-         The rocker is pinned at arm_link5 (C, this joint origin) and
-         its free end tracks the pad's middle hole via the mimic
-         relationship.  Positions match the original yahboomcar
-         URDF which works correctly in RViz. -->
+         keeps the pad parallel through the whole grip range. -->
     <xacro:common_link_no_collision name="rlink3" material="Green" path="X3plus">
         <inertial>
@@ -457,5 +452,5 @@
     </xacro:common_link_no_collision>
     <xacro:continuous_joint name="rlink_joint3" parent="arm_link5" child="rlink3" xyz="-0.0035 -0.0045 -0.0505"
-                      rpy="0 -${pi/2} 0" mimic="1"/>
+                      rpy="0 -${pi/2} 0" mimic="-1"/>
     <xacro:common_link_no_collision name="llink1" material="Green" path="X3plus">
         <inertial>
@@ -475,5 +470,5 @@
     </xacro:common_link>
     <xacro:continuous_joint name="llink_joint2" parent="llink1" child="llink2" xyz="0.03 0.00065104 0" rpy="0 0 0"
-                      mimic="1"/>
+                      mimic="-1"/>
     <!-- llink3 / llink_joint3: LEFT 4-bar ROCKER, mirror of the right side.
          Mirror of the right rocker with Y axis flipped.  mimic=-1 so the
@@ -587,29 +582,16 @@
             <initial_position>0</initial_position>
         </plugin>
-        <!-- ==================== MIMIC GRIPPER FINGER CONTROLLERS ====================
-              Ignition Fortress does NOT enforce URDF <mimic>. To make the fingers
-              actually open/close in Gazebo (not just visually in RViz/RSP), we
-              attach a low-gain JointPositionController to each of the 3 mimic
-              joints (rlink_joint2, llink_joint1, llink_joint2). The
-              gripper_mimic_relay node fans out /grip_joint_cmd_pos to each
-              /<mimic>_cmd_pos topic with the URDF multiplier baked in.
-              Finger inertias are bumped to 1e-5 (above) and gravity is disabled
-              on the finger links (below) so these tiny PID loops stay stable. -->
-        <!-- MIMIC GRIPPER FINGER CONTROLLERS (5 mimic joints).
-             rlink_joint3 and llink_joint3 are the 4-bar COUPLERS (rockers).
-             All five share the same low-gain PID: p_gain=10, i_gain=0.0 (any
-             integral winds up against the joint limit and freezes/splays the
-             finger), d_gain=0.3.  The couplers keep the pads parallel and make
-             the four-bar visually complete. -->
+        <!-- MIMIC GRIPPER FINGER CONTROLLERS (5 mimic joints, min-gain).
+             Low gains (P=2.0, cmd_max=1.0 N.m) — enough to move the 1g
+             finger links without creating a PID bidding war against
+             grip_joint (P=50, cmd_max=2.5).  The relay's 10 rad/s ramp
+             rate ensures the reference never jumps. -->
         <plugin filename="ignition-gazebo-joint-position-controller-system"
                 name="ignition::gazebo::systems::JointPositionController">
             <joint_name>llink_joint1</joint_name>
             <topic>/llink_joint1_cmd_pos</topic>
-            <p_gain>50.0</p_gain> <i_gain>0.0</i_gain>  <d_gain>2.0</d_gain>
-            <i_max>0.2</i_max> <i_min>-0.2</i_min>
-            <cmd_max>2.5</cmd_max> <cmd_min>-2.5</cmd_min>
-            <!-- mimic=-1: at master=-1.54 the mimic should be at +1.54.
-                 Setting initial to the correct mimic value avoids the
-                 sim-start jump that visibly "detaches" the pad. -->
+            <p_gain>2.0</p_gain> <i_gain>0.0</i_gain>  <d_gain>0.2</d_gain>
+            <i_max>0.1</i_max> <i_min>-0.1</i_min>
+            <cmd_max>1.0</cmd_max> <cmd_min>-1.0</cmd_min>
             <initial_position>0</initial_position>
         </plugin>
@@ -618,7 +600,7 @@
             <joint_name>llink_joint2</joint_name>
             <topic>/llink_joint2_cmd_pos</topic>
-            <p_gain>50.0</p_gain> <i_gain>0.0</i_gain>  <d_gain>2.0</d_gain>
-            <i_max>0.2</i_max> <i_min>-0.2</i_min>
-            <cmd_max>2.5</cmd_max> <cmd_min>-2.5</cmd_min>
+            <p_gain>2.0</p_gain> <i_gain>0.0</i_gain>  <d_gain>0.2</d_gain>
+            <i_max>0.1</i_max> <i_min>-0.1</i_min>
+            <cmd_max>1.0</cmd_max> <cmd_min>-1.0</cmd_min>
             <initial_position>0</initial_position>
         </plugin>
@@ -627,8 +609,7 @@
             <joint_name>llink_joint3</joint_name>
             <topic>/llink_joint3_cmd_pos</topic>
-            <p_gain>50.0</p_gain> <i_gain>0.0</i_gain>  <d_gain>2.0</d_gain>
-            <i_max>0.2</i_max> <i_min>-0.2</i_min>
-            <cmd_max>2.5</cmd_max> <cmd_min>-2.5</cmd_min>
-            <!-- mimic=-1: at master=-1.54 the mimic should be at +1.54. -->
+            <p_gain>2.0</p_gain> <i_gain>0.0</i_gain>  <d_gain>0.2</d_gain>
+            <i_max>0.1</i_max> <i_min>-0.1</i_min>
+            <cmd_max>1.0</cmd_max> <cmd_min>-1.0</cmd_min>
             <initial_position>0</initial_position>
         </plugin>
@@ -637,8 +618,7 @@
             <joint_name>rlink_joint2</joint_name>
             <topic>/rlink_joint2_cmd_pos</topic>
-            <p_gain>50.0</p_gain> <i_gain>0.0</i_gain>  <d_gain>2.0</d_gain>
-            <i_max>0.2</i_max> <i_min>-0.2</i_min>
-            <cmd_max>2.5</cmd_max> <cmd_min>-2.5</cmd_min>
-            <!-- mimic=-1: at master=-1.54 the mimic should be at +1.54. -->
+            <p_gain>2.0</p_gain> <i_gain>0.0</i_gain>  <d_gain>0.2</d_gain>
+            <i_max>0.1</i_max> <i_min>-0.1</i_min>
+            <cmd_max>1.0</cmd_max> <cmd_min>-1.0</cmd_min>
             <initial_position>0</initial_position>
         </plugin>
@@ -647,7 +627,7 @@
             <joint_name>rlink_joint3</joint_name>
             <topic>/rlink_joint3_cmd_pos</topic>
-            <p_gain>50.0</p_gain> <i_gain>0.0</i_gain>  <d_gain>2.0</d_gain>
-            <i_max>0.2</i_max> <i_min>-0.2</i_min>
-            <cmd_max>2.5</cmd_max> <cmd_min>-2.5</cmd_min>
+            <p_gain>2.0</p_gain> <i_gain>0.0</i_gain>  <d_gain>0.2</d_gain>
+            <i_max>0.1</i_max> <i_min>-0.1</i_min>
+            <cmd_max>1.0</cmd_max> <cmd_min>-1.0</cmd_min>
             <initial_position>0</initial_position>
         </plugin>
